File: Fichiers Kicad/Projet_ControlledEnvironment/Projet_ControlledEnvironment.kicad_pcb (KiCad board)
At the start: 2 copper layers, 140 x 85 mm, 42 parts, among them J201 Pi 40-Pin Connector, J401 Conn_01x02, J402 Conn_01x02, J403 Conn_01x02, J404 Conn_01x04, J405 Conn_01x02, J406 Conn_01x02, J407 Conn_01x02, J408 Conn_01x02, J409 Conn_01x02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

Commit message: GUI Added et Modif Kicad
Connections:
- U201 pad 1: LED_FAN_OUT -> /Mainblock Core/GPIO18
- U201 pad 2: /Mainblock Core/GPIO18 -> LED_FAN_OUT
- U202 pad 1: BOITIER_FAN_OUT -> /Mainblock Core/GPIO12
- U202 pad 2: /Mainblock Core/GPIO12 -> BOITIER_FAN_OUT
- U203 pad 1: EXT_OPT_FAN_OUT -> /Mainblock Core/GPIO19
- U203 pad 2: /Mainblock Core/GPIO19 -> EXT_OPT_FAN_OUT
- U209 pad 1: 100W_LED- -> /Mainblock Core/GPIO13
- U209 pad 2: /Mainblock Core/GPIO13 -> 100W_LED-
Routing:
- net /Mainblock Core/GPIO19: track 109.3 -> 112.9 mm
- net 100W_LED-: track 14.5 -> 15.8 mm
- net /Mainblock Core/GPIO18: track 66.7 -> 68.0 mm
- net /Mainblock Core/GPIO12: track 85.6 -> 86.8 mm
- net BOITIER_FAN_OUT: track 32.3 -> 31.2 mm
- net /Mainblock Core/GPIO13: track 20.2 -> 19.1 mm
- net EXT_OPT_FAN_OUT: track 31.6 -> 30.7 mm
- net LED_FAN_OUT: track 33.2 -> 32.5 mm
